Commit message: finished step 5

File: Step5/table_macro.xacro (robot description, xacro)
@@ -64,5 +64,5 @@
       <parent link="${parent}" />
       <child link="table_top" />
-      <origin xyz="0 0 ${table_height + table_thickness}" rpy="0 0 0" />
+      <origin xyz="0 0 0" rpy="${pi} 0 0" />
     </joint>
   <!-- Base Link, Table Top -->

File: Step5/table_on_robot.urdf.xacro (robot description, xacro)
@@ -6,9 +6,9 @@
     <xacro:include filename="rrbot_macro.xacro" />
     <link name="world" />
-    <xacro:table parent="world">
-        <origin xyz="0 0 1" rpy="0 0 0" />
-    </xacro:table>
-    <xacro:table parent="tool_joint">
+    <xacro:rrbot parent="world">
         <origin xyz="0 0 0" rpy="0 0 0" />
+    </xacro:rrbot>
+    <xacro:table parent="tool0">
+        <origin xyz="0 0 0" rpy="${pi} 0 0" />
     </xacro:table>
 </robot>
