Commit message: completed step 6

File: ws1/src/rrbot_on_table_description/urdf/rrbot_on_table.urdf.xacro (robot description, xacro)
@@ -5,14 +5,15 @@
   <xacro:include filename="$(find rrbot_on_table_description)/urdf/common/inertials.xacro"/>
   <xacro:include filename="$(find rrbot_on_table_description)/urdf/common/materials.xacro"/>
+  <xacro:include filename="$(find table_description)/urdf/table/table_macro.xacro"/>
   <xacro:include filename="$(find rrbot_description)/urdf/rrbot/rrbot_macro.xacro"/>
-  <xacro:include filename="$(find table_description)/urdf/table/table_macro.xacro"/>
+  <xacro:arg name="table_prefix" default="table_" />
   <!-- create link fixed to the "world" -->
   <link name="world" />
   <!-- Load robot's macro with parameters -->
   <!-- set prefix if multiple robots are used -->
-  <xacro:table prefix="table_" parent="world" >
+  <xacro:table prefix="$(arg table_prefix)" parent="world" >
     <origin xyz="0 0 1" rpy="0 0 0" />          <!-- position robot in the world -->
   </xacro:table>
-  <xacro:rrbot prefix="rrbot_" parent="table_top" >
+  <xacro:rrbot prefix="rrbot_" parent="$(arg table_prefix)table_top" >
     <origin xyz="0 0 0" rpy="0 0 0" />          <!-- position robot in the world -->
   </xacro:rrbot>

File: ws1/src/table_description/urdf/table/table_macro.xacro (robot description, xacro)
@@ -41,21 +41,21 @@
     <!-- Attach the legs to the table_top using fixed joints -->
     <joint name="${prefix}leg1_joint" type="fixed">
-      <parent link="table_top" />
-      <child link="leg1" />
+      <parent link="${prefix}table_top" />
+      <child link="${prefix}leg1" />
       <origin xyz="${table_length/2 - leg_radius} ${table_width/2 - leg_radius} ${-table_thickness}" rpy="0 0 0" />
     </joint>
     <joint name="${prefix}leg2_joint" type="fixed">
-      <parent link="table_top" />
-      <child link="leg2" />
+      <parent link="${prefix}table_top" />
+      <child link="${prefix}leg2" />
       <origin xyz="${-table_length/2 + leg_radius} ${table_width/2 - leg_radius} ${-table_thickness}" rpy="0 0 0" />
     </joint>
     <joint name="${prefix}leg3_joint" type="fixed">
-      <parent link="table_top" />
-      <child link="leg3" />
+      <parent link="${prefix}table_top" />
+      <child link="${prefix}leg3" />
       <origin xyz="${-table_length/2 + leg_radius} ${-table_width/2 + leg_radius} ${-table_thickness}" rpy="0 0 0" />
     </joint>
     <joint name="${prefix}leg4_joint" type="fixed">
-      <parent link="table_top" />
-      <child link="leg4" />
+      <parent link="${prefix}table_top" />
+      <child link="${prefix}leg4" />
       <origin xyz="${table_length/2 - leg_radius} ${-table_width/2 + leg_radius} ${-table_thickness}" rpy="0 0 0" />
     </joint>
@@ -63,5 +63,5 @@
     <joint name="${prefix}table_top_joint" type="fixed">
       <parent link="${parent}" />
-      <child link="table_top" />
+      <child link="${prefix}table_top" />
       <origin xyz="0 0 ${table_height + table_thickness}" rpy="0 0 0" />
     </joint>
